File: DE0-Nano-SoC_LED.sch (KiCad schematic (older format))
At the start: 6 parts, among them J1 Conn_02x08_Odd_Even, J2 Conn_02x08_Odd_Even, J3 Conn_02x20_Odd_Even, J4 Conn_02x20_Odd_Even, U1 74HC245, U2 74HC245

Commit message: still in connectors placement phase
Parts:
- added J10, J11, J12, J13, J14, J15, J8, J9: Conn_01x01, Mounting_Holes:MountingHole_3.2mm_M3_ISO7380_Pad, symbol Conn_01x01
- added J16: Conn_01x10, Pin_Headers:Pin_Header_Straight_1x10_Pitch2.54mm, symbol Conn_01x10
- added J17, J19: Conn_01x08, Pin_Headers:Pin_Header_Straight_1x08_Pitch2.54mm, symbol Conn_01x08
- added J18: Conn_01x06, Pin_Headers:Pin_Header_Straight_1x06_Pitch2.54mm, symbol Conn_01x06
- added J5, J6, J7: Conn_02x08_Odd_Even, Connectors_Multicomp:Multicomp_MC9A12-1634_2x08x2.54mm_Straight, symbol Conn_02x08_Odd_Even
- added RN1, RN2: R_Pack04, Resistors_SMD:R_Array_Concave_4x0402, symbol R_Pack04
Connections:
- net labels added: 3V3, 9V, VCC
- wire segments 11 -> 85
Other:
- moved on the sheet: J2, J3, J4, U2

Commit message: half of the components are almost placed
Parts:
- added C1, C10, C2, C3, C4, C5, C6, C7, C8, C9: 0.1, Capacitors_SMD:C_0402_NoSilk, symbol C
- added C11, C12, C13, C14, C15, C16, C17, C18, C19, C20: 0.01, Capacitors_SMD:C_0402_NoSilk, symbol C
- added RN10, RN11, RN12, RN13, RN14, RN15, RN16, RN17, RN18, RN19, RN20, RN3, RN4, RN5, RN6, RN7, RN8, RN9: R_Pack04, Resistors_SMD:R_Array_Concave_4x0402, symbol R_Pack04
- added U10, U3, U4, U5, U6, U7, U8, U9: 74HC245, SMD_Packages:SSOP-20, symbol 74HC245
Connections:
- net labels added: A_1_1, A_2_1, A_3_1, A_4_1, A_5_1, A__1, B1_1, B1_1_1, B1_2, B1_2_1, B1_3, B1_3_1, B1_4, B1_4_1, B1_5, B1_5_1, B2_1, B2_1_1, B2_2, B2_2_1, B2_3, B2_3_1, B2_4, B2_4_1, B2_5, B2_5_1, B_1_1, B_2_1, B_3_1, B_4_1, B_5_1, B__1, CLK_1_1, CLK_2_1, CLK_3_1, CLK_4_1, CLK_5_1, CLK__1, C_1_1, C_2_1, C_3_1, C_4_1, C_5_1, C__1, D_1_1, D_2_1, D_3_1, D_4_1, D_5_1, D__1, G1_1, G1_1_1, G1_2, G1_2_1, G1_3, G1_3_1, G1_4, G1_4_1, G1_5, G1_5_1, G2_1, G2_1_1, G2_2, G2_2_1, G2_3, G2_3_1, G2_4, G2_4_1, G2_5, G2_5_1, LAT_1_1, LAT_2_1, LAT_3_1, LAT_4_1, LAT_5_1, LAT__1, OE_1_1, OE_2_1, OE_3_1, OE_4_1, OE_5_1, OE__1, R1_1, R1_1_1, R1_2, R1_2_1, R1_3, R1_3_1, R1_4, R1_4_1, R1_5, R1_5_1, R2_1, R2_1_1, R2_2, R2_2_1, R2_3, R2_3_1, R2_4, R2_4_1, R2_5, R2_5_1
- wire segments 85 -> 445
Other:
- moved on the sheet: J1, J10, J11, J12, J13, J14, J15, J16, J17, J18, J19, J2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

Commit message: a lot of progress on pcb
Changed lines of the file:
@@
 R1_3_1
 Text Label 9250 5950 0    60   ~ 0
-R2_3
+B2_3
 Text Label 9250 5850 0    60   ~ 0
 G2_3
@@
 B1_3
 Text Label 2750 8150 0    60   ~ 0
+B1_3
+Text Label 4150 8150 0    60   ~ 0
 G1_3
-Text Label 4150 8150 0    60   ~ 0
-B1_3
 Text Label 2750 8250 0    60   ~ 0
+R2_3
+Text Label 4150 8250 0    60   ~ 0
 R1_3
-Text Label 4150 8250 0    60   ~ 0
-R2_3
 Text Label 2750 8350 0    60   ~ 0
+B2_3
+Text Label 4150 8350 0    60   ~ 0
 G2_3
-Text Label 4150 8350 0    60   ~ 0
-B2_3
 Wire Wire Line
 	3300 8450 2650 8450
@@
 	3800 8450 4500 8450
 Text Label 2750 8450 0    60   ~ 0
+B1_4
+Text Label 4150 8450 0    60   ~ 0
 G1_4
-Text Label 4150 8450 0    60   ~ 0
-B1_4
 Wire Wire Line
 	3300 8850 2650 8850
@@
 	3300 9050 2650 9050
 Text Label 2750 8850 0    60   ~ 0
+B1_5
+Text Label 4150 8850 0    60   ~ 0
 G1_5
-Text Label 4150 8850 0    60   ~ 0
-B1_5
 Text Label 2750 8950 0    60   ~ 0
+G2_5
+Text Label 4150 8950 0    60   ~ 0
 R1_5
-Text Label 4150 8950 0    60   ~ 0
+Text Label 2750 9050 0    60   ~ 0
+B2_5
+Text Label 4150 9050 0    60   ~ 0
 R2_5
-Text Label 2750 9050 0    60   ~ 0
-G2_5
-Text Label 4150 9050 0    60   ~ 0
-B2_5
 Wire Wire Line
 	3800 8650 4500 8650
@@
 	3300 8750 2650 8750
 Text Label 2750 8650 0    60   ~ 0
+R2_4
+Text Label 4150 8650 0    60   ~ 0
 R1_4
-Text Label 4150 8650 0    60   ~ 0
-R2_4
 Text Label 2750 8750 0    60   ~ 0
+B2_4
+Text Label 4150 8750 0    60   ~ 0
 G2_4
-Text Label 4150 8750 0    60   ~ 0
-B2_4
 Wire Wire Line
 	2750 5450 2850 5450

Commit message: more progress on pcb
Connections:
- wire segments 445 -> 446
Changed lines of the file:
@@
 Wire Wire Line
 	1750 7900 2250 7900
-Text Label 1950 7900 0    60   ~ 0
-OE__1
 Text Label 4150 8050 0    60   ~ 0
 B__1
@@
 Wire Wire Line
 	13700 9050 13700 9100
+Wire Wire Line
+	1750 7700 2250 7700
+Text Label 1950 7700 0    60   ~ 0
+OE__1
 $EndSCHEMATC

Commit message: small improvemets in pcb
Parts:
- added C21: C, Capacitors_SMD:C_1210, symbol C
Connections:
- wire segments 446 -> 493
Changed lines of the file:
@@
 	18250 5450 18350 5450
 Wire Wire Line
-	2850 5550 2800 5550
+	2750 5550 2850 5550
 Connection ~ 2800 6250
 Wire Wire Line
-	2850 5650 2800 5650
+	2250 5650 2850 5650
 Connection ~ 2800 5650
 Wire Wire Line
-	6800 5550 6750 5550
+	6700 5550 6800 5550
 Connection ~ 6750 6250
 Wire Wire Line
-	6800 5650 6750 5650
+	6200 5650 6800 5650
 Connection ~ 6750 5650
 Wire Wire Line
-	10650 5550 10600 5550
+	10550 5550 10650 5550
 Connection ~ 10600 6250
 Wire Wire Line
-	10650 5650 10600 5650
+	10050 5650 10650 5650
 Connection ~ 10600 5650
 Wire Wire Line
-	14500 5550 14450 5550
+	14400 5550 14500 5550
 Connection ~ 14450 6250
 Wire Wire Line
-	14500 5650 14450 5650
+	13900 5650 14500 5650
 Connection ~ 14450 5650
 Wire Wire Line
-	18350 5550 18300 5550
+	18250 5550 18350 5550
 Connection ~ 18300 6250
 Wire Wire Line
-	18350 5650 18300 5650
+	17750 5650 18350 5650
 Connection ~ 18300 5650
 $Comp
@@
 $EndComp
 Wire Wire Line
-	2850 3750 2800 3750
-Wire Wire Line
-	2800 3750 2800 3600
+	2750 3750 2850 3750
+Wire Wire Line
+	2800 3600 2800 3750
 $Comp
 L GND #PWR036
@@
 $EndComp
 Wire Wire Line
-	6750 3750 6700 3750
-Wire Wire Line
-	6700 3750 6700 3650
-Wire Wire Line
-	10650 3750 10600 3750
-Wire Wire Line
-	10600 3750 10600 3650
-Wire Wire Line
-	14500 3750 14450 3750
-Wire Wire Line
-	14450 3750 14450 3650
-Wire Wire Line
-	18350 3750 18300 3750
-Wire Wire Line
-	18300 3750 18300 3650
+	6650 3750 6750 3750
+Wire Wire Line
+	6700 3650 6700 3750
+Wire Wire Line
+	10550 3750 10650 3750
+Wire Wire Line
+	10600 3650 10600 3750
+Wire Wire Line
+	14400 3750 14500 3750
+Wire Wire Line
+	14450 3650 14450 3750
+Wire Wire Line
+	18250 3750 18350 3750
+Wire Wire Line
+	18300 3650 18300 3750
 $Comp
 L C C1
@@
 Text Label 1950 7700 0    60   ~ 0
 OE__1
+Connection ~ 2800 5550
+Wire Wire Line
+	1800 5550 2350 5550
+Wire Wire Line
+	2300 5550 2300 5650
+Connection ~ 2300 5650
+Wire Wire Line
+	1850 5650 1800 5650
+Wire Wire Line
+	1800 5650 1800 5550
+Connection ~ 2300 5550
+Connection ~ 2800 3750
+Wire Wire Line
+	2350 3750 2200 3750
+Wire Wire Line
+	2200 3750 2200 3600
+Wire Wire Line
+	2200 3600 2700 3600
+Wire Wire Line
+	2700 3600 2700 3650
+Wire Wire Line
+	2700 3650 2800 3650
+Connection ~ 2800 3650
+Connection ~ 6750 5550
+Wire Wire Line
+	5750 5550 6300 5550
+Wire Wire Line
+	6250 5550 6250 5650
+Connection ~ 6250 5650
+Wire Wire Line
+	5800 5650 5750 5650
+Wire Wire Line
+	5750 5650 5750 5550
+Connection ~ 6250 5550
+Connection ~ 10600 5550
+Wire Wire Line
+	9600 5550 10150 5550
+Wire Wire Line
+	10100 5550 10100 5650
+Connection ~ 10100 5650
+Wire Wire Line
+	9650 5650 9600 5650
+Wire Wire Line
+	9600 5650 9600 5550
+Connection ~ 10100 5550
+Connection ~ 6700 3750
+Wire Wire Line
+	6250 3750 6200 3750
+Wire Wire Line
+	6200 3750 6200 3650
+Wire Wire Line
+	6200 3650 6600 3650
+Wire Wire Line
+	6600 3650 6600 3700
+Wire Wire Line
+	6600 3700 6700 3700
+Connection ~ 6700 3700
+Connection ~ 10600 3750
+Wire Wire Line
+	10150 3750 10100 3750
+Wire Wire Line
+	10100 3750 10100 3650
+Wire Wire Line
+	10100 3650 10550 3650
+Wire Wire Line
+	10550 3650 10550 3700
+Wire Wire Line
+	10550 3700 10600 3700
+Connection ~ 10600 3700
+Connection ~ 14450 3750
+Wire Wire Line
+	14000 3750 13950 3750
+Wire Wire Line
+	13950 3750 13950 3650
+Wire Wire Line
+	13950 3650 14350 3650
+Wire Wire Line
+	14350 3650 14350 3700
+Wire Wire Line
+	14350 3700 14450 3700
+Connection ~ 14450 3700
+Connection ~ 14450 5550
+Wire Wire Line
+	13450 5550 14000 5550
+Wire Wire Line
+	13950 5550 13950 5650
+Connection ~ 13950 5650
+Wire Wire Line
+	13500 5650 13450 5650
+Wire Wire Line
+	13450 5650 13450 5550
+Connection ~ 13950 5550
+Connection ~ 18300 3750
+Wire Wire Line
+	17850 3750 17750 3750
+Wire Wire Line
+	17750 3750 17750 3650
+Wire Wire Line
+	17750 3650 18200 3650
+Wire Wire Line
+	18200 3650 18200 3700
+Wire Wire Line
+	18200 3700 18300 3700
+Connection ~ 18300 3700
+Connection ~ 18300 5550
+Wire Wire Line
+	17250 5550 17850 5550
+Wire Wire Line
+	17800 5550 17800 5650
+Connection ~ 17800 5650
+Wire Wire Line
+	17350 5650 17250 5650
+Wire Wire Line
+	17250 5650 17250 5550
+Connection ~ 17800 5550
+$Comp
+L GND #PWR080
+U 1 1 5A2A092E
+P 13250 8650
+F 0 "#PWR080" H 13250 8400 50  0001 C CNN
+F 1 "GND" H 13250 8500 50  0000 C CNN
+F 2 "" H 13250 8650 50  0001 C CNN
+F 3 "" H 13250 8650 50  0001 C CNN
+	1    13250 8650
+	1    0    0    -1
+$EndComp
+Wire Wire Line
+	13250 8650 13250 8600
+$Comp
+L VCC #PWR081
+U 1 1 5A2A105D
+P 13250 8250
+F 0 "#PWR081" H 13250 8100 50  0001 C CNN
+F 1 "VCC" H 13250 8400 50  0000 C CNN
+F 2 "" H 13250 8250 50  0001 C CNN
+F 3 "" H 13250 8250 50  0001 C CNN
+	1    13250 8250
+	1    0    0    -1
+$EndComp
+Wire Wire Line
+	13250 8300 13250 8250
+$Comp
+L C C21
+U 1 1 5A2A0757
+P 13250 8450
+F 0 "C21" H 13275 8550 50  0000 L CNN
+F 1 "C" H 13275 8350 50  0000 L CNN
+F 2 "Capacitors_SMD:C_1210" H 13288 8300 50  0001 C CNN
+F 3 "" H 13250 8450 50  0001 C CNN
+	1    13250 8450
+	1    0    0    -1
+$EndComp
 $EndSCHEMATC

Commit message: final version of half board
Parts:
- removed J10, J12, J13, J9: Conn_01x01, Mounting_Holes:MountingHole_3.2mm_M3_ISO7380_Pad, symbol Conn_01x01
- removed J18: Conn_01x06, Pin_Headers:Pin_Header_Straight_1x06_Pitch2.54mm, symbol Conn_01x06
- removed J19: Conn_01x08, Pin_Headers:Pin_Header_Straight_1x08_Pitch2.54mm, symbol Conn_01x08
- removed J4: Conn_02x20_Odd_Even, Pin_Headers:Pin_Header_Straight_2x20_Pitch2.54mm, symbol Conn_02x20_Odd_Even
Connections:
- net labels removed: 9V
- wire segments 493 -> 467

Commit message: back to full board
Parts:
- added J10: Conn_01x08, Pin_Headers:Pin_Header_Straight_1x08_Pitch2.54mm, symbol Conn_01x08
- added J12, J13, J18, J19: Conn_01x01, Mounting_Holes:MountingHole_3.2mm_M3_ISO7380_Pad, symbol Conn_01x01
- added J4: Conn_02x20_Odd_Even, Pin_Headers:Pin_Header_Straight_2x20_Pitch2.54mm, symbol Conn_02x20_Odd_Even
- added J9: Conn_01x06, Pin_Headers:Pin_Header_Straight_1x06_Pitch2.54mm, symbol Conn_01x06
Connections:
- net labels added: A__2, B1_10, B1_6, B1_7, B1_8, B1_9, B2_10, B2_6, B2_7, B2_8, B2_9, B__2, CLK__2, C__2, D__2, G1_10, G1_6, G1_7, G1_8, G1_9, G2_10, G2_6, G2_7, G2_8, G2_9, LAT__2, R1_10, R1_6, R1_7, R1_8, R1_9, R2_10, R2_6, R2_7, R2_8, R2_9
- wire segments 467 -> 512
Other:
- moved on the sheet: C1, C10, C11, C12, C13, C14, C15, C16, C17, C18, C19, C2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

Commit message: pin rename
Changed lines of the file:
@@
 	5650 6700 5000 6700
 Text Label 6500 6600 0    60   ~ 0
-R2_10
+R2_6
 Text Label 6500 6700 0    60   ~ 0
-B2_10
+B2_6
 Wire Wire Line
 	5650 6800 5000 6800
@@
 	5650 7100 5000 7100
 Text Label 6500 6800 0    60   ~ 0
-B1_9
+B1_7
 Text Label 6500 6900 0    60   ~ 0
-R2_9
+R2_7
 Text Label 5100 7100 0    60   ~ 0
-G2_9
+G2_7
 Text Label 6500 7100 0    60   ~ 0
-B2_9
+B2_7
 Text Label 5100 7500 0    60   ~ 0
 B1_8
@@
 	6150 7800 6850 7800
 Text Label 5100 7800 0    60   ~ 0
-B1_7
+B1_9
 Text Label 6500 7800 0    60   ~ 0
-G1_7
+G1_9
 Wire Wire Line
 	5650 8200 5000 8200
@@
 	5650 8400 5000 8400
 Text Label 5100 8200 0    60   ~ 0
-B1_6
+B1_10
 Text Label 6500 8200 0    60   ~ 0
-G1_6
+G1_10
 Text Label 5100 8300 0    60   ~ 0
-G2_6
+G2_10
 Text Label 6500 8300 0    60   ~ 0
-R1_6
+R1_10
 Text Label 5100 8400 0    60   ~ 0
-B2_6
+B2_10
 Text Label 6500 8400 0    60   ~ 0
-R2_6
+R2_10
 Wire Wire Line
 	6150 8000 6850 8000
@@
 	5650 8100 5000 8100
 Text Label 5100 8000 0    60   ~ 0
-R2_7
+R2_9
 Text Label 6500 8000 0    60   ~ 0
+R1_9
+Text Label 5100 8100 0    60   ~ 0
+B2_9
+Text Label 6500 8100 0    60   ~ 0
+G2_9
+Text Label 6500 6500 0    60   ~ 0
+B1_6
+Text Label 5100 6900 0    60   ~ 0
 R1_7
-Text Label 5100 8100 0    60   ~ 0
-B2_7
-Text Label 6500 8100 0    60   ~ 0
-G2_7
-Text Label 6500 6500 0    60   ~ 0
-B1_10
-Text Label 5100 6900 0    60   ~ 0
-R1_9
 Text Label 5100 6800 0    60   ~ 0
-G1_9
+G1_7
 Text Label 5100 6700 0    60   ~ 0
-G2_10
+G2_6
 Text Label 5100 6600 0    60   ~ 0
-R1_10
+R1_6
 Text Label 5100 6500 0    60   ~ 0
-G1_10
+G1_6
 $Comp
 L Conn_01x06 J9
