File: DE0-Nano-SoC_LED.sch (KiCad schematic (older format))
At the start: 127 parts, among them J1 Conn_02x08_Odd_Even, J10 Conn_01x08, J11 Conn_01x01, J12 Conn_01x01, J13 Conn_01x01, J14 Conn_01x01, J15 Conn_01x01, J16 Conn_01x10, J17 Conn_01x08, J18 Conn_01x01, J19 Conn_01x01, J2 Conn_02x08_Odd_Even, J20 Conn_02x08_Odd_Even, J21 Conn_02x08_Odd_Even, J22 Conn_02x08_Odd_Even, J23 Conn_02x08_Odd_Even, J24 Conn_02x08_Odd_Even, J3 Conn_02x20_Odd_Even, J4 Conn_02x20_Odd_Even, J5 Conn_02x08_Odd_Even, J6 Conn_02x08_Odd_Even, J7 Conn_02x08_Odd_Even, J8 Conn_01x01, J9 Conn_01x06, U1 74HC245, U10 74HC245, U11 74HC245, U12 74HC245, U13 74HC245, U14 74HC245, U15 74HC245, U16 74HC245, U17 74HC245, U18 74HC245, U19 74HC245, U2 74HC245, U20 74HC245, U3 74HC245, U4 74HC245, U5 74HC245, U6 74HC245, U7 74HC245, U8 74HC245, U9 74HC245

Commit message: new connectors
Parts:
- removed J?: Conn_01x05, symbol Conn_01x05
- added J25: Conn_01x10, Pin_Headers:Pin_Header_Straight_1x10_Pitch2.54mm, symbol Conn_01x10
- added J26, J27: Conn_01x06, Pin_Headers:Pin_Header_Straight_1x06_Pitch2.54mm, symbol Conn_01x06
Connections:
- net labels added: ADC_IN0, ADC_IN1, ADC_IN2, ADC_IN3, ADC_IN4, ADC_IN5, FPGA_AF13, FPGA_AG10, FPGA_AG13
- wire segments 948 -> 960

Commit message: what should I add to the board?
Parts:
- added J28: Conn_01x10, Pin_Headers:Pin_Header_Straight_1x10_Pitch2.54mm, symbol Conn_01x10
Connections:
- net labels added: FPGA_AG11, FPGA_AG16, FPGA_AH11, FPGA_AH12, FPGA_AH9
- wire segments 960 -> 982
Other:
- moved on the sheet: J25
Changed lines of the file:
@@
 	1    0    0    -1
 $EndComp
-Text Label 2000 7050 0    60   ~ 0
-OE__1
 $Comp
 L GND #PWR076
@@
 	13750 8400 13750 8450
 Wire Wire Line
-	1800 7050 2300 7050
+	1800 7050 2450 7050
 Connection ~ 2850 4900
 Wire Wire Line
@@
 L Conn_01x10 J25
 U 1 1 5A6A3D1E
-P 800 6850
-F 0 "J25" H 800 7350 50  0000 C CNN
-F 1 "Conn_01x10" H 800 6250 50  0000 C CNN
-F 2 "Pin_Headers:Pin_Header_Straight_1x10_Pitch2.54mm" H 800 6850 50  0001 C CNN
-F 3 "" H 800 6850 50  0001 C CNN
-	1    800  6850
+P 700 6850
+F 0 "J25" H 700 7350 50  0000 C CNN
+F 1 "Conn_01x10" H 700 6250 50  0000 C CNN
+F 2 "Pin_Headers:Pin_Header_Straight_1x10_Pitch2.54mm" H 700 6850 50  0001 C CNN
+F 3 "" H 700 6850 50  0001 C CNN
+	1    700  6850
 	-1   0    0    -1
 $EndComp
@@
 Text Label 2000 9400 0    60   ~ 0
 FPGA_AG10
+$Comp
+L Conn_01x10 J28
+U 1 1 5A69DE2E
+P 700 8100
+F 0 "J28" H 700 8600 50  0000 C CNN
+F 1 "Conn_01x10" H 700 7500 50  0000 C CNN
+F 2 "Pin_Headers:Pin_Header_Straight_1x10_Pitch2.54mm" H 700 8100 50  0001 C CNN
+F 3 "" H 700 8100 50  0001 C CNN
+	1    700  8100
+	-1   0    0    -1
+$EndComp
+$Comp
+L GND #PWR0158
+U 1 1 5A69E18E
+P 1000 8700
+F 0 "#PWR0158" H 1000 8450 50  0001 C CNN
+F 1 "GND" H 1000 8550 50  0000 C CNN
+F 2 "" H 1000 8700 50  0001 C CNN
+F 3 "" H 1000 8700 50  0001 C CNN
+	1    1000 8700
+	1    0    0    -1
+$EndComp
+Wire Wire Line
+	1000 8600 900  8600
+Wire Wire Line
+	1000 8300 1000 8700
+Wire Wire Line
+	900  8500 1000 8500
+Connection ~ 1000 8600
+Wire Wire Line
+	900  8400 1000 8400
+Connection ~ 1000 8500
+Wire Wire Line
+	900  8300 1000 8300
+Connection ~ 1000 8400
+$Comp
+L VCC #PWR0159
+U 1 1 5A6A18EA
+P 1100 7350
+F 0 "#PWR0159" H 1100 7200 50  0001 C CNN
+F 1 "VCC" H 1100 7500 50  0000 C CNN
+F 2 "" H 1100 7350 50  0001 C CNN
+F 3 "" H 1100 7350 50  0001 C CNN
+	1    1100 7350
+	0    1    1    0
+$EndComp
+Wire Wire Line
+	900  7150 1000 7150
+Wire Wire Line
+	1000 7150 1000 7350
+Wire Wire Line
+	900  7350 1100 7350
+Wire Wire Line
+	900  7250 1000 7250
+Connection ~ 1000 7250
+Connection ~ 1000 7350
+Wire Wire Line
+	1800 6450 2450 6450
+Wire Wire Line
+	1800 6550 2450 6550
+Wire Wire Line
+	1800 6850 2450 6850
+Wire Wire Line
+	1800 6950 2450 6950
+Text Label 1850 6450 0    60   ~ 0
+FPGA_AG11
+Text Label 1850 6550 0    60   ~ 0
+FPGA_AH9
+Text Label 1950 6850 0    60   ~ 0
+FPGA_AH12
+Text Label 1950 6950 0    60   ~ 0
+FPGA_AH11
+Wire Wire Line
+	900  6450 1400 6450
+Wire Wire Line
+	900  6550 1400 6550
+Wire Wire Line
+	900  6850 1400 6850
+Wire Wire Line
+	900  6950 1400 6950
+Wire Wire Line
+	900  7050 1400 7050
+Wire Wire Line
+	1800 7150 2450 7150
+Text Label 1950 7050 0    60   ~ 0
+FPGA_AG16
+Text Label 1950 7150 0    60   ~ 0
+OE__1
+Text Label 950  6450 0    60   ~ 0
+FPGA_AG11
+Text Label 950  6550 0    60   ~ 0
+FPGA_AH9
+$Comp
+L GND #PWR?
+U 1 1 5A69ECAC
+P 1000 6650
+F 0 "#PWR?" H 1000 6400 50  0001 C CNN
+F 1 "GND" H 1000 6500 50  0000 C CNN
+F 2 "" H 1000 6650 50  0001 C CNN
+F 3 "" H 1000 6650 50  0001 C CNN
+	1    1000 6650
+	0    -1   -1   0
+$EndComp
+Wire Wire Line
+	900  6750 950  6750
+Wire Wire Line
+	950  6750 950  6650
+Wire Wire Line
+	900  6650 1000 6650
+Connection ~ 950  6650
+Text Label 950  6850 0    60   ~ 0
+FPGA_AH12
+Text Label 950  6950 0    60   ~ 0
+FPGA_AH11
+Text Label 950  7050 0    60   ~ 0
+FPGA_AG16
 $EndSCHEMATC

Commit message: final 1.1 version
Parts:
- added J29, J30: Conn_01x01, Mounting_Holes:MountingHole_3.2mm_M3_ISO7380_Pad, symbol Conn_01x01
- added J31: Conn_01x04, Pin_Headers:Pin_Header_Straight_1x04_Pitch2.54mm, symbol Conn_01x04
Connections:
- wire segments 982 -> 990
Changed lines of the file:
@@
 	16700 14350 16600 14350
 Wire Wire Line
-	16600 14350 16600 15350
+	16600 13650 16600 15350
 Wire Wire Line
 	16700 15250 16600 15250
@@
 FPGA_AH9
 $Comp
-L GND #PWR?
+L GND #PWR0160
 U 1 1 5A69ECAC
 P 1000 6650
-F 0 "#PWR?" H 1000 6400 50  0001 C CNN
+F 0 "#PWR0160" H 1000 6400 50  0001 C CNN
 F 1 "GND" H 1000 6500 50  0000 C CNN
 F 2 "" H 1000 6650 50  0001 C CNN
@@
 Text Label 950  7050 0    60   ~ 0
 FPGA_AG16
+$Comp
+L Conn_01x01 J30
+U 1 1 5A7D94D1
+P 16900 13950
+F 0 "J30" H 16900 14050 50  0000 C CNN
+F 1 "Conn_01x01" H 16900 13850 50  0000 C CNN
+F 2 "Mounting_Holes:MountingHole_3.2mm_M3_ISO7380_Pad" H 16900 13950 50  0001 C CNN
+F 3 "" H 16900 13950 50  0001 C CNN
+	1    16900 13950
+	1    0    0    -1
+$EndComp
+$Comp
+L Conn_01x01 J29
+U 1 1 5A7D9682
+P 16900 13650
+F 0 "J29" H 16900 13750 50  0000 C CNN
+F 1 "Conn_01x01" H 16900 13550 50  0000 C CNN
+F 2 "Mounting_Holes:MountingHole_3.2mm_M3_ISO7380_Pad" H 16900 13650 50  0001 C CNN
+F 3 "" H 16900 13650 50  0001 C CNN
+	1    16900 13650
+	1    0    0    -1
+$EndComp
+Wire Wire Line
+	16700 13950 16600 13950
+Connection ~ 16600 14350
+Wire Wire Line
+	16700 13650 16600 13650
+Connection ~ 16600 13950
+$Comp
+L Conn_01x04 J31
+U 1 1 5A7DDDD0
+P 7850 8050
+F 0 "J31" H 7850 8250 50  0000 C CNN
+F 1 "Conn_01x04" H 7850 7750 50  0000 C CNN
+F 2 "Pin_Headers:Pin_Header_Straight_1x04_Pitch2.54mm" H 7850 8050 50  0001 C CNN
+F 3 "" H 7850 8050 50  0001 C CNN
+	1    7850 8050
+	-1   0    0    1
+$EndComp
+$Comp
+L GND #PWR0161
+U 1 1 5A7DE3A3
+P 8150 8250
+F 0 "#PWR0161" H 8150 8000 50  0001 C CNN
+F 1 "GND" H 8150 8100 50  0000 C CNN
+F 2 "" H 8150 8250 50  0001 C CNN
+F 3 "" H 8150 8250 50  0001 C CNN
+	1    8150 8250
+	1    0    0    -1
+$EndComp
+Wire Wire Line
+	8050 8150 8150 8150
+Wire Wire Line
+	8150 8050 8150 8250
+Wire Wire Line
+	8050 8050 8150 8050
+Connection ~ 8150 8150
+Wire Wire Line
+	8050 7950 8600 7950
+Wire Wire Line
+	8050 7850 8150 7850
+Wire Wire Line
+	8150 7850 8150 7950
+Connection ~ 8150 7950
+Text Label 8300 7950 0    60   ~ 0
+3V3
 $EndSCHEMATC
